Commit message: Added Xtion sample robot

File: common_sensors/urdf/sensors/xtion_xtended_stand.urdf.xacro (robot description, xacro)
@@ -56,7 +56,7 @@
 		</link>
 	</xacro:macro>
-	<xacro:macro name="xtion_plate" params="parent x_loc y_loc z_loc">
+	<xacro:macro name="xtion_plate" params="parent x_loc y_loc z_loc angle">
 		<joint name="xtion_plate_joint" type="fixed">
-			<origin xyz="${x_loc} ${y_loc} ${z_loc}" rpy="0 -0.7853 0" />
+            <origin xyz="${x_loc} ${y_loc} ${z_loc}" rpy="0 ${angle} 0" />
 			<parent link="${parent}" />
 			<child link="xtion_plate_link" />
@@ -85,5 +85,6 @@
 	<xacro:property name="plate_thickness" value="0.006" />
 	<xacro:property name="xtion_mount_z" value="0.035" />
-	<xacro:macro name="xtion_stand" params="parent">
+	<!--xacro:property name="tilting_angle" value="-0.7853" /-->
+	<xacro:macro name="xtion_stand" params="parent tilting_angle">
 		<xacro:xtion_standoff number="1" parent="${parent}" x_loc="0" y_loc="-0.1" z_loc="${cyl_height/2}" height="${cyl_height}"/>
 		<xacro:xtion_standoff number="2" parent="${parent}" x_loc="0" y_loc="0.1" z_loc="${cyl_height/2}" height="${cyl_height}"/>
@@ -93,5 +94,5 @@
 		<xacro:xtion_standoff number="5" parent="${parent}" x_loc="0" y_loc="-0.1" z_loc="${cyl_height*1.5+plate_thickness}" height="${cyl_height}"/>
 		<xacro:xtion_standoff number="6" parent="${parent}" x_loc="0" y_loc="0.1" z_loc="${cyl_height*1.5+plate_thickness}" height="${cyl_height}"/>
-		<xacro:xtion_plate parent="standoff_6_link" x_loc="0" y_loc="-0.1" z_loc="${cyl_height/2+xtion_mount_z}"/>
+        <xacro:xtion_plate parent="standoff_6_link" x_loc="0" y_loc="-0.1" z_loc="${cyl_height/2+xtion_mount_z}" angle="${tilting_angle}"/>
 		<xacro:sensor_xtion parent="xtion_plate_link" camera_name="jaco_xtion">
 			<origin xyz="0 0 ${xtion_height/2+plate_thickness/2}" rpy="0 0 3.14159" />
