Commit message: update readme

File: common_sensors/urdf/sensors/kinect.urdf.xacro (robot description, xacro)
@@ -41,5 +41,5 @@
 			 <origin xyz="0 0 0" rpy="0 0 ${M_PI/2}"/>
 				<geometry>
-				<mesh filename="package://common_sensors/meshes/kinect.dae"/>
+				<mesh filename="package://common_sensors/meshes/sensors/kinect.dae"/>
 				</geometry>
 			</visual>

Commit message: Update kinect: fixed bug reported in issue #2

File: common_sensors/urdf/sensors/kinect.urdf.xacro (robot description, xacro)
@@ -33,5 +33,5 @@
 		</link>
 		<joint name="camera_joint" type="fixed">
-			<origin xyz="-0.031 ${-cam_y} -0.016" rpy="0 0 0"/>
+			<origin xyz="-0.031 ${-cam_py} -0.016" rpy="0 0 0"/>
 			<parent link="camera_rgb_frame"/>
 			<child link="camera_link"/>
@@ -60,5 +60,5 @@
 		 (Hence, don't publish them additionally!) -->
 		<joint name="camera_depth_joint" type="fixed">
-			<origin xyz="0 ${2 * -cam_y} 0" rpy="0 0 0" />
+			<origin xyz="0 ${2 * -cam_py} 0" rpy="0 0 0" />
 			<parent link="camera_rgb_frame" />
 			<child link="camera_depth_frame" />

File: common_sensors/urdf/sensors/kinect_properties.urdf.xacro (robot description, xacro)
@@ -2,12 +2,11 @@
 <root>
   <!--
-    These properties must be observed by any machine
-	translation and rotation of camera from the tabletop
+	  Translation and rotation of camera from its base link
    -->
-	<property name="cam_px" value="-0.4" />
-	<property name="cam_py" value="1.0" />
+	<property name="cam_px" value="0" />
+	<property name="cam_py" value="0" />
 	<property name="cam_pz" value="0" />
-	<property name="cam_or" value="-1.57079632679" />
-	<property name="cam_op" value="0.4" />
+	<property name="cam_or" value="0" />
+	<property name="cam_op" value="0" />
 	<property name="cam_oy" value="0" />
 </root>
