Commit message: Further improvements to Kinect2 models

File: common_sensors/urdf/sensors/kinect2.gazebo.xacro (robot description, xacro)
@@ -1,5 +1,5 @@
 <?xml version="1.0"?>
 <robot xmlns:xacro="http://ros.org/wiki/xacro">
-<xacro:macro name="kinect2_ir_gazebo_v0" params="link_name frame_name camera_name">
+<xacro:macro name="kinect2_ir_gazebo" params="link_name frame_name camera_name">
   <gazebo reference="${link_name}">
     <sensor type="depth" name="${name}_ir_sensor">
@@ -45,5 +45,5 @@
   </gazebo>
 </xacro:macro>
-<xacro:macro name="kinect2_rgb_gazebo_v0" params="link_name frame_name camera_name">
+<xacro:macro name="kinect2_rgb_gazebo" params="link_name frame_name camera_name">
   <gazebo reference="${link_name}">
     <sensor type="depth" name="${name}_rgb_sensor">

File: common_sensors/urdf/sensors/kinect2.urdf.xacro (robot description, xacro)
@@ -6,5 +6,5 @@
   <xacro:property name="ir_depth_rgb_offset_y" value="0.01"/> <!-- FIXME: what is this offset? -->
   <!-- Kinect2 and mount assembly -->
-  <xacro:macro name="kinect2_v0" params="name parent *origin">
+  <xacro:macro name="kinect2" params="name parent *origin">
     <joint name="${name}_kinect2_joint" type="fixed">
       <xacro:insert_block name="origin" />
@@ -72,5 +72,5 @@
     <link name="${name}_kinect2_ir_optical_frame"/>
     <!-- gazebo extensions -->
-    <xacro:kinect2_ir_gazebo_v0 link_name="${name}_kinect2_ir_link" frame_name="${name}_kinect2_ir_optical_frame" camera_name="head_mount_kinect2" />
+    <xacro:kinect2_ir_gazebo link_name="${name}_kinect2_ir_link" frame_name="${name}_kinect2_ir_optical_frame" camera_name="head_mount_kinect2" />
     <!-- kinect2 rgb sensor physical attachment -->
     <joint name="${name}_kinect2_rgb_joint" type="fixed">
@@ -110,5 +110,5 @@
     <link name="${name}_kinect2_rgb_optical_frame"/>
     <!-- gazebo extensions -->
-    <xacro:kinect2_rgb_gazebo_v0 link_name="${name}_kinect2_rgb_link" frame_name="${name}_kinect2_rgb_optical_frame" camera_name="head_mount_kinect2" />
+    <xacro:kinect2_rgb_gazebo link_name="${name}_kinect2_rgb_link" frame_name="${name}_kinect2_rgb_optical_frame" camera_name="head_mount_kinect2" />
   </xacro:macro>
 </robot>

Commit message: :wrench: Updates kinect2 configuration values

File: common_sensors/urdf/sensors/kinect2.gazebo.xacro (robot description, xacro)
@@ -1,90 +1,90 @@
 <?xml version="1.0"?>
 <robot xmlns:xacro="http://www.ros.org/wiki/xacro">
-<xacro:macro name="kinect2_ir_gazebo" params="link_name frame_name camera_name">
-  <gazebo reference="${link_name}">
-    <sensor type="depth" name="${name}_ir_sensor">
-      <always_on>true</always_on>
-      <update_rate>1.0</update_rate>
-      <camera>
-        <horizontal_fov>${57.0*M_PI/180.0}</horizontal_fov>
-        <image>
-          <format>L8</format>
-          <width>640</width>
-          <height>480</height>
-        </image>
-        <clip>
-          <near>0.01</near>
-          <far>5</far>
-        </clip>
-      </camera>
-      <plugin name="${link_name}_controller" filename="libgazebo_ros_openni_kinect.so">
-        <baseline>0.2</baseline>
-        <alwaysOn>true</alwaysOn>
-        <updateRate>1.0</updateRate>
-        <cameraName>${camera_name}_ir</cameraName>
-        <imageTopicName>/${camera_name}/ir/image_raw</imageTopicName>
-        <cameraInfoTopicName>/${camera_name}/ir/camera_info</cameraInfoTopicName>
-        <depthImageTopicName>/${camera_name}/depth/image_raw</depthImageTopicName>
-        <depthImageCameraInfoTopicName>/${camera_name}/depth/camera_info</depthImageCameraInfoTopicName>
-        <pointCloudTopicName>/${camera_name}/depth/points</pointCloudTopicName>
-        <frameName>${frame_name}</frameName>
-        <pointCloudCutoff>0.5</pointCloudCutoff>
-        <distortionK1>0.00000001</distortionK1>
-        <distortionK2>0.00000001</distortionK2>
-        <distortionK3>0.00000001</distortionK3>
-        <distortionT1>0.00000001</distortionT1>
-        <distortionT2>0.00000001</distortionT2>
-        <CxPrime>0</CxPrime>
-        <Cx>0</Cx>
-        <Cy>0</Cy>
-        <focalLength>0</focalLength>
-        <hackBaseline>0</hackBaseline>
-      </plugin>
-    </sensor>
-    <material value="Gazebo/Red" />
-  </gazebo>
-</xacro:macro>
-<xacro:macro name="kinect2_rgb_gazebo" params="link_name frame_name camera_name">
-  <gazebo reference="${link_name}">
-    <sensor type="depth" name="${name}_rgb_sensor">
-      <always_on>true</always_on>
-      <update_rate>1.0</update_rate>
-      <camera>
-        <horizontal_fov>${57.0*M_PI/180.0}</horizontal_fov>
-        <image>
-          <format>B8G8R8</format>
-          <width>640</width>
-          <height>480</height>
-        </image>
-        <clip>
-          <near>0.01</near>
-          <far>5</far>
-        </clip>
-      </camera>
-      <plugin name="${link_name}_controller" filename="libgazebo_ros_openni_kinect.so">
-        <alwaysOn>true</alwaysOn>
-        <updateRate>1.0</updateRate>
-        <cameraName>${camera_name}_rgb</cameraName>
-        <imageTopicName>/${camera_name}/rgb/image_raw</imageTopicName>
-        <cameraInfoTopicName>/${camera_name}/rgb/camera_info</cameraInfoTopicName>
-        <depthImageTopicName>/${camera_name}/depth/image_raw</depthImageTopicName>
-        <depthImageCameraInfoTopicName>/${camera_name}/depth/camera_info</depthImageCameraInfoTopicName>
-        <pointCloudTopicName>/${camera_name}/depth_registered/points</pointCloudTopicName>
-        <frameName>${frame_name}</frameName>
-        <pointCloudCutoff>0.5</pointCloudCutoff>
-        <distortionK1>0.00000001</distortionK1>
-        <distortionK2>0.00000001</distortionK2>
-        <distortionK3>0.00000001</distortionK3>
-        <distortionT1>0.00000001</distortionT1>
-        <distortionT2>0.00000001</distortionT2>
-        <CxPrime>0</CxPrime>
-        <Cx>0</Cx>
-        <Cy>0</Cy>
-        <focalLength>0</focalLength>
-        <hackBaseline>0</hackBaseline>
-      </plugin>
-    </sensor>
-    <material value="Gazebo/Red" />
-  </gazebo>
-</xacro:macro>
+  <xacro:macro name="kinect2_ir_gazebo" params="link_name frame_name camera_name">
+    <gazebo reference="${link_name}">
+      <sensor type="depth" name="${name}_ir_sensor">
+        <always_on>true</always_on>
+        <update_rate>1.0</update_rate>
+        <camera>
+          <horizontal_fov>${57.0*M_PI/180.0}</horizontal_fov>
+          <image>
+            <format>L8</format>
+            <width>640</width>
+            <height>480</height>
+          </image>
+          <clip>
+            <near>0.01</near>
+            <far>5</far>
+          </clip>
+        </camera>
+        <plugin name="${link_name}_controller" filename="libgazebo_ros_openni_kinect.so">
+          <baseline>0.2</baseline>
+          <alwaysOn>true</alwaysOn>
+          <updateRate>1.0</updateRate>
+          <cameraName>${camera_name}_ir</cameraName>
+          <imageTopicName>/${camera_name}/ir/image_raw</imageTopicName>
+          <cameraInfoTopicName>/${camera_name}/ir/camera_info</cameraInfoTopicName>
+          <depthImageTopicName>/${camera_name}/depth/image_raw</depthImageTopicName>
+          <depthImageCameraInfoTopicName>/${camera_name}/depth/camera_info</depthImageCameraInfoTopicName>
+          <pointCloudTopicName>/${camera_name}/depth/points</pointCloudTopicName>
+          <frameName>${frame_name}</frameName>
+          <pointCloudCutoff>0.5</pointCloudCutoff>
+          <distortionK1>0.00000001</distortionK1>
+          <distortionK2>0.00000001</distortionK2>
+          <distortionK3>0.00000001</distortionK3>
+          <distortionT1>0.00000001</distortionT1>
+          <distortionT2>0.00000001</distortionT2>
+          <CxPrime>0</CxPrime>
+          <Cx>0</Cx>
+          <Cy>0</Cy>
+          <focalLength>0</focalLength>
+          <hackBaseline>0</hackBaseline>
+        </plugin>
+      </sensor>
+      <material value="Gazebo/Red" />
+    </gazebo>
+  </xacro:macro>
+  <xacro:macro name="kinect2_rgb_gazebo" params="link_name frame_name camera_name">
+    <gazebo reference="${link_name}">
+      <sensor type="depth" name="${name}_rgb_sensor">
+        <always_on>true</always_on>
+        <update_rate>1.0</update_rate>
+        <camera>
+          <horizontal_fov>${57.0*M_PI/180.0}</horizontal_fov>
+          <image>
+            <format>B8G8R8</format>
+            <width>640</width>
+            <height>480</height>
+          </image>
+          <clip>
+            <near>0.01</near>
+            <far>5</far>
+          </clip>
+        </camera>
+        <plugin name="${link_name}_controller" filename="libgazebo_ros_openni_kinect.so">
+          <alwaysOn>true</alwaysOn>
+          <updateRate>1.0</updateRate>
+          <cameraName>${camera_name}_rgb</cameraName>
+          <imageTopicName>/${camera_name}/rgb/image_raw</imageTopicName>
+          <cameraInfoTopicName>/${camera_name}/rgb/camera_info</cameraInfoTopicName>
+          <depthImageTopicName>/${camera_name}/depth/image_raw</depthImageTopicName>
+          <depthImageCameraInfoTopicName>/${camera_name}/depth/camera_info</depthImageCameraInfoTopicName>
+          <pointCloudTopicName>/${camera_name}/depth_registered/points</pointCloudTopicName>
+          <frameName>${frame_name}</frameName>
+          <pointCloudCutoff>0.5</pointCloudCutoff>
+          <distortionK1>0.00000001</distortionK1>
+          <distortionK2>0.00000001</distortionK2>
+          <distortionK3>0.00000001</distortionK3>
+          <distortionT1>0.00000001</distortionT1>
+          <distortionT2>0.00000001</distortionT2>
+          <CxPrime>0</CxPrime>
+          <Cx>0</Cx>
+          <Cy>0</Cy>
+          <focalLength>0</focalLength>
+          <hackBaseline>0</hackBaseline>
+        </plugin>
+      </sensor>
+      <material value="Gazebo/Red" />
+    </gazebo>
+  </xacro:macro>
 </robot>

File: common_sensors/urdf/sensors/kinect2.urdf.xacro (robot description, xacro)
@@ -4,19 +4,18 @@
   <xacro:include filename="$(find common_sensors)/urdf/sensors/kinect2_properties.urdf.xacro" />
   <xacro:include filename="$(find common_sensors)/urdf/common_properties.urdf.xacro" />
-  <xacro:property name="ir_depth_rgb_offset_y" value="0.01"/> <!-- FIXME: what is this offset? -->
+  <xacro:property name="ir_depth_rgb_offset_y" value="0.01"/>
+  <!-- FIXME: what is this offset? -->
   <!-- Kinect2 and mount assembly -->
-  <xacro:macro name="kinect2" params="name parent *origin">
-    <joint name="${name}_kinect2_joint" type="fixed">
+  <xacro:macro name="kinect2" params="name camera_name parent *origin">
+    <joint name="${name}_joint" type="fixed">
       <xacro:insert_block name="origin" />
       <parent link="${parent}"/>
-      <child link="${name}_kinect2_link"/>
+      <child link="${name}_link"/>
     </joint>
-    <link name="${name}_kinect2_link">
+    <link name="${name}_link">
       <inertial>
         <mass value="0.1"/>
         <origin xyz="0 0 0" rpy="0 0 0"/>
-        <inertia ixx="0.01"  ixy="0.0"  ixz="0.0"
-                 iyy="0.01"  iyz="0.0"
-                 izz="0.01" />
+        <inertia ixx="0.01" ixy="0.0" ixz="0.0" iyy="0.01" iyz="0.0" izz="0.01" />
       </inertial>
       <visual>
@@ -37,16 +36,14 @@
     </link>
     <!-- kinect2 ir sensor physical attachment -->
-    <joint name="${name}_kinect2_ir_joint" type="fixed">
+    <joint name="${name}_ir_joint" type="fixed">
       <origin xyz="-0.032267 -0.0475 0.155" rpy="0 0 0"/>
-      <parent link="${name}_kinect2_link"/>
-      <child link="${name}_kinect2_ir_link"/>
+      <parent link="${name}_link"/>
+      <child link="${name}_ir_link"/>
     </joint>
-    <link name="${name}_kinect2_ir_link">
+    <link name="${name}_ir_link">
       <inertial>
         <mass value="0.1" />
         <origin xyz="0 0 0" rpy="0 0 0"/>
-        <inertia ixx="0.01"  ixy="0.0"  ixz="0.0"
-                 iyy="0.01"  iyz="0.0"
-                 izz="0.01" />
+        <inertia ixx="0.01" ixy="0.0" ixz="0.0" iyy="0.01" iyz="0.0" izz="0.01" />
       </inertial>
       <visual>
@@ -64,30 +61,26 @@
     </link>
     <!-- kinect2 ir sensor frame -->
-    <joint name="${name}_kinect2_ir_optical_frame_joint" type="fixed">
-      <origin xyz="${cal_kinect_x}                  ${cal_kinect_y+ir_depth_rgb_offset_y} ${cal_kinect_z}"
-              rpy="${-M_PI/2+cal_kinect_roll}       ${0.0+cal_kinect_pitch}               ${-M_PI/2+cal_kinect_yaw}" />
-      <parent link="${name}_kinect2_ir_link"/>
-      <child link="${name}_kinect2_ir_optical_frame"/>
+    <joint name="${name}_ir_optical_frame_joint" type="fixed">
+      <origin xyz="${cal_kinect_x}                  ${cal_kinect_y+ir_depth_rgb_offset_y} ${cal_kinect_z}" rpy="${-M_PI/2+cal_kinect_roll}       ${0.0+cal_kinect_pitch}               ${-M_PI/2+cal_kinect_yaw}" />
+      <parent link="${name}_ir_link"/>
+      <child link="${name}_ir_optical_frame"/>
     </joint>
-    <link name="${name}_kinect2_ir_optical_frame"/>
+    <link name="${name}_ir_optical_frame"/>
     <!-- gazebo extensions -->
-    <xacro:kinect2_ir_gazebo link_name="${name}_kinect2_ir_link" frame_name="${name}_kinect2_ir_optical_frame" camera_name="head_mount_kinect2" />
+    <xacro:kinect2_ir_gazebo link_name="${name}_ir_link" frame_name="${name}_ir_optical_frame" camera_name="${camera_name}" />
     <!-- kinect2 rgb sensor physical attachment -->
-    <joint name="${name}_kinect2_rgb_joint" type="fixed">
+    <joint name="${name}_rgb_joint" type="fixed">
       <origin xyz="0 -0.05175 0" rpy="0 0 0"/>
-      <parent link="${name}_kinect2_ir_link"/>
-      <child link="${name}_kinect2_rgb_link"/>
+      <parent link="${name}_ir_link"/>
+      <child link="${name}_rgb_link"/>
     </joint>
-    <link name="${name}_kinect2_rgb_link" >
+    <link name="${name}_rgb_link">
       <inertial>
         <mass value="0.1" />
         <origin xyz="0 0 0" rpy="0 0 0"/>
-        <inertia ixx="0.01"  ixy="0.0"  ixz="0.0"
-                 iyy="0.01"  iyz="0.0"
-                 izz="0.01" />
+        <inertia ixx="0.01" ixy="0.0" ixz="0.0" iyy="0.01" iyz="0.0" izz="0.01" />
       </inertial>
       <visual>
-        <origin xyz="${cal_kinect_x}            ${cal_kinect_y}                 ${cal_kinect_z}"
-                rpy="${-M_PI/2+cal_kinect_roll} ${0.0+cal_kinect_pitch}         ${-M_PI/2+cal_kinect_yaw}" />
+        <origin xyz="${cal_kinect_x}            ${cal_kinect_y}                 ${cal_kinect_z}" rpy="${-M_PI/2+cal_kinect_roll} ${0.0+cal_kinect_pitch}         ${-M_PI/2+cal_kinect_yaw}" />
         <geometry>
           <sphere radius="0.0005"/>
@@ -102,13 +95,12 @@
     </link>
     <!-- kinect2 rgb sensor frame -->
-    <joint name="${name}_kinect2_rgb_optical_frame_joint" type="fixed">
-      <origin xyz="${cal_kinect_x}            ${cal_kinect_y}                 ${cal_kinect_z}"
-              rpy="${-M_PI/2+cal_kinect_roll} ${0.0+cal_kinect_pitch}         ${-M_PI/2+cal_kinect_yaw}" />
-      <parent link="${name}_kinect2_rgb_link"/>
-      <child link="${name}_kinect2_rgb_optical_frame"/>
+    <joint name="${name}_rgb_optical_frame_joint" type="fixed">
+      <origin xyz="${cal_kinect_x}            ${cal_kinect_y}                 ${cal_kinect_z}" rpy="${-M_PI/2+cal_kinect_roll} ${0.0+cal_kinect_pitch}         ${-M_PI/2+cal_kinect_yaw}" />
+      <parent link="${name}_rgb_link"/>
+      <child link="${name}_rgb_optical_frame"/>
     </joint>
-    <link name="${name}_kinect2_rgb_optical_frame"/>
+    <link name="${name}_rgb_optical_frame"/>
     <!-- gazebo extensions -->
-    <xacro:kinect2_rgb_gazebo link_name="${name}_kinect2_rgb_link" frame_name="${name}_kinect2_rgb_optical_frame" camera_name="head_mount_kinect2" />
+    <xacro:kinect2_rgb_gazebo link_name="${name}_rgb_link" frame_name="${name}_rgb_optical_frame" camera_name="${camera_name}" />
   </xacro:macro>
 </robot>

File: common_sensors/urdf/sensors/xtion_gazebo.urdf.xacro (robot description, xacro)
@@ -1,4 +1,5 @@
 <?xml version="1.0"?>
-<robot name="xtion_gazebo" xmlns:xacro="http://ros.org/wiki/xacro">
+<robot name="xtion_gazebo"
+  xmlns:xacro="http://ros.org/wiki/xacro">
   <!-- Microsoft Kinect / ASUS Xtion PRO Live for simulation -->
   <xacro:macro name="xtion_sim_3dsensor" params="camera_name">
